File: Eagle/AddSub.sch (EAGLE design)
At the start: 238 parts, among them Q1 310mA/60V/1.6Ω, Q10 310mA/60V/1.6Ω, Q100 310mA/60V/1.6Ω, Q101 310mA/60V/1.6Ω, Q102 310mA/60V/1.6Ω, Q103 310mA/60V/1.6Ω, Q104 310mA/60V/1.6Ω, Q105 310mA/60V/1.6Ω, Q106 310mA/60V/1.6Ω, Q107 310mA/60V/1.6Ω, Q108 310mA/60V/1.6Ω, Q109 310mA/60V/1.6Ω, Q11 310mA/60V/1.6Ω, Q110 310mA/60V/1.6Ω, Q111 310mA/60V/1.6Ω, Q112 310mA/60V/1.6Ω, Q113 310mA/60V/1.6Ω, Q114 310mA/60V/1.6Ω, Q115 310mA/60V/1.6Ω, Q116 310mA/60V/1.6Ω, Q117 310mA/60V/1.6Ω, Q118 310mA/60V/1.6Ω, Q119 310mA/60V/1.6Ω, Q12 310mA/60V/1.6Ω, Q120 310mA/60V/1.6Ω, Q121 310mA/60V/1.6Ω, Q122 310mA/60V/1.6Ω, Q123 310mA/60V/1.6Ω, Q124 310mA/60V/1.6Ω, Q125 310mA/60V/1.6Ω, Q126 310mA/60V/1.6Ω, Q127 310mA/60V/1.6Ω, Q13 310mA/60V/1.6Ω, Q134 310mA/60V/1.6Ω, Q135 310mA/60V/1.6Ω, Q136 310mA/60V/1.6Ω, Q137 310mA/60V/1.6Ω, Q138 310mA/60V/1.6Ω, Q139 310mA/60V/1.6Ω, Q14 310mA/60V/1.6Ω, Q140 310mA/60V/1.6Ω, Q148 310mA/60V/1.6Ω, Q149 310mA/60V/1.6Ω, Q15 310mA/60V/1.6Ω, Q150 310mA/60V/1.6Ω, Q151 310mA/60V/1.6Ω, Q152 310mA/60V/1.6Ω, Q153 310mA/60V/1.6Ω, Q154 310mA/60V/1.6Ω, Q16 310mA/60V/1.6Ω, Q162 310mA/60V/1.6Ω, Q163 310mA/60V/1.6Ω, Q164 310mA/60V/1.6Ω, Q165 310mA/60V/1.6Ω, Q166 310mA/60V/1.6Ω, Q167 310mA/60V/1.6Ω, Q168 310mA/60V/1.6Ω, Q17 310mA/60V/1.6Ω, Q176 310mA/60V/1.6Ω, Q177 310mA/60V/1.6Ω, Q178 310mA/60V/1.6Ω, Q179 310mA/60V/1.6Ω, Q18 310mA/60V/1.6Ω, Q180 310mA/60V/1.6Ω, Q181 310mA/60V/1.6Ω, Q182 310mA/60V/1.6Ω, Q19 310mA/60V/1.6Ω, Q2 310mA/60V/1.6Ω, Q20 310mA/60V/1.6Ω, Q21 310mA/60V/1.6Ω, Q22 310mA/60V/1.6Ω, Q23 310mA/60V/1.6Ω, Q24 310mA/60V/1.6Ω, Q25 310mA/60V/1.6Ω, Q26 310mA/60V/1.6Ω, Q27 310mA/60V/1.6Ω, Q28 310mA/60V/1.6Ω, Q29 310mA/60V/1.6Ω, Q3 310mA/60V/1.6Ω, Q30 310mA/60V/1.6Ω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

Commit message: Rerouted for SOT23
Parts:
- removed Q134, Q135, Q136, Q137, Q138, Q139, Q140, Q151, Q152, Q153, Q154, Q162, Q176, Q32, Q36, Q40, Q50, Q51, Q52, Q62: 310mA/60V/1.6Ω, SparkFun-DiscreteSemi:MOSFET-NCH-2N7002PW
- removed R20, R30, R31, R32, R68, R69, R70, R71, R79, R84, R85, R92, R93: (no value), SparkFun-Resistors:RESISTOR0805
- added Q128, Q129, Q130, Q131, Q132, Q133, Q141, Q142, Q143, Q144, Q145, Q146, Q147, Q155, Q156, Q157, Q158, Q159, Q169, Q183: 310mA/60V/1.6Ω, XSNOR:NMOSREFLOW
- added R66, R67, R72, R73, R74, R75, R80, R81, R82, R88, R89, R96, R97: (no value), XSNOR:RESISTOR0805
- Q1, Q10, Q100, Q101, Q102, Q103, Q104, Q105, Q106, Q107, Q108, Q109, Q11, Q110, Q111, Q112, Q113, Q114, Q115, Q116, Q117, Q118, Q119, Q12, Q120, Q121, Q122, Q123, Q124, Q125, Q126, Q127, Q13, Q14, Q148, Q149, Q15, Q150, Q16, Q163, Q164, Q165, Q166, Q167, Q168, Q17, Q177, Q178, Q179, Q18, Q180, Q181, Q182, Q19, Q2, Q20, Q21, Q22, Q23, Q24, Q25, Q26, Q27, Q28, Q29, Q3, Q30, Q31, Q33, Q34, Q35, Q37, Q38, Q39, Q4, Q41, Q42, Q43, Q44, Q45, Q46, Q47, Q48, Q49, Q5, Q53, Q54, Q55, Q56, Q57, Q58, Q59, Q6, Q60, Q61, Q63, Q64, Q65, Q66, Q67, Q68, Q69, Q7, Q70, Q71, Q72, Q73, Q74, Q75, Q76, Q77, Q78, Q79, Q8, Q80, Q81, Q82, Q83, Q84, Q85, Q86, Q87, Q88, Q89, Q9, Q90, Q91, Q92, Q93, Q94, Q95, Q96, Q97, Q98, Q99: device SparkFun-DiscreteSemi:MOSFET-NCH-2N7002PW -> XSNOR:NMOSREFLOW
- R1, R10, R11, R12, R13, R14, R15, R16, R17, R18, R19, R2, R21, R22, R23, R24, R25, R26, R27, R28, R29, R3, R33, R34, R35, R36, R37, R38, R39, R4, R40, R41, R42, R43, R44, R45, R46, R47, R48, R49, R5, R50, R51, R52, R53, R54, R55, R56, R57, R58, R59, R6, R60, R61, R62, R63, R64, R65, R7, R76, R77, R78, R8, R86, R87, R9, R94, R95: device SparkFun-Resistors:RESISTOR0805 -> XSNOR:RESISTOR0805
Connections:
- removed net N$1: Q134.D, Q136.G, R68.1
- removed net N$2: Q73.D, Q76.D, Q80.G, Q85.G, R37.1
- removed net N$4: Q148.D, Q150.G, R76.1
- removed net N1: Q137.D, Q138.D, Q139.G, R70.1
- removed net N10: Q28.D, Q32.D, Q36.G, Q50.G, R16.1
- removed net N11: Q51.D, Q63.D, Q72.G, R31.1
- removed net N13: Q36.D, Q40.D, Q51.G, Q52.G, Q62.G, R20.1
- removed net N14: Q16.G, Q23.G, Q4.D, Q64.G, Q8.D, R4.1
- removed net N18: Q165.D, Q166.D, Q167.G, R86.1
- removed net N19: Q163.D, Q164.D, Q168.G, R85.1
- removed net N2: Q135.D, Q136.D, Q140.G, R69.1
- removed net N22: Q14.D, Q22.D, Q31.G, R10.1
- removed net N23: Q13.D, Q21.D, Q27.G, R9.1
- removed net N24: Q27.D, Q31.D, Q35.G, Q47.G, R15.1
- removed net N25: Q48.D, Q60.D, Q71.G, R28.1
- removed net N26: Q47.D, Q59.D, Q67.G, R27.1
- removed net N27: Q35.D, Q39.D, Q48.G, Q49.G, Q59.G, R19.1
- removed net N28: Q14.G, Q21.G, Q3.D, Q61.G, Q7.D, R3.1
- removed net N29: Q179.D, Q180.D, Q181.G, R94.1
- removed net N30: Q177.D, Q178.D, Q182.G, R93.1
- removed net N36: Q12.D, Q20.D, Q30.G, R8.1
- removed net N37: Q11.D, Q19.D, Q26.G, R7.1
- removed net N38: Q26.D, Q30.D, Q34.G, Q44.G, R14.1
- removed net N39: Q45.D, Q57.D, Q70.G, R25.1
- removed net N40: Q44.D, Q56.D, Q66.G, R24.1
- removed net N41: Q34.D, Q38.D, Q45.G, Q46.G, Q56.G, R18.1
- removed net N42: Q12.G, Q19.G, Q2.D, Q58.G, Q6.D, R2.1
- removed net N5: Q151.D, Q152.D, Q153.G, R78.1
- removed net N50: Q10.D, Q18.D, Q29.G, R6.1
- removed net N51: Q17.D, Q25.G, Q9.D, R5.1
- removed net N52: Q25.D, Q29.D, Q33.G, Q41.G, R13.1
- removed net N53: Q42.D, Q54.D, Q69.G, R22.1
- removed net N54: Q41.D, Q53.D, Q65.G, R21.1
- removed net N55: Q33.D, Q37.D, Q42.G, Q43.G, Q53.G, R17.1
- removed net N56: Q1.D, Q10.G, Q17.G, Q5.D, Q55.G, R1.1
- removed net N6: Q149.D, Q150.D, Q154.G, R77.1
- removed net N64: Q84.D, Q90.D, Q96.G, R45.1
- removed net N65: Q83.D, Q89.D, Q93.G, R44.1
- removed net N66: Q109.G, Q93.D, Q96.D, Q99.G, R48.1
- removed net N67: Q110.D, Q119.D, Q126.G, R59.1
- removed net N68: Q109.D, Q118.D, Q123.G, R58.1
- removed net N69: Q102.D, Q110.G, Q111.G, Q118.G, Q99.D, R51.1
- removed net N70: Q120.G, Q75.D, Q78.D, Q84.G, Q89.G, R39.1
- removed net N78: Q82.D, Q88.D, Q95.G, R43.1
- removed net N79: Q81.D, Q87.D, Q92.G, R42.1
- removed net N8: Q16.D, Q24.D, Q32.G, R12.1
- removed net N80: Q106.G, Q92.D, Q95.D, Q98.G, R47.1
- removed net N81: Q107.D, Q116.D, Q125.G, R56.1
- removed net N82: Q106.D, Q115.D, Q122.G, R55.1
- removed net N83: Q101.D, Q107.G, Q108.G, Q115.G, Q98.D, R50.1
- removed net N84: Q117.G, Q74.D, Q77.D, Q82.G, Q87.G, R38.1
- removed net N9: Q15.D, Q23.D, Q28.G, R11.1
- removed net N92: Q80.D, Q86.D, Q94.G, R41.1
- removed net N93: Q79.D, Q85.D, Q91.G, R40.1
- removed net N94: Q103.G, Q91.D, Q94.D, Q97.G, R46.1
- removed net N95: Q104.D, Q113.D, Q124.G, R53.1
- removed net N96: Q103.D, Q112.D, Q121.G, R52.1
- removed net N97: Q100.D, Q104.G, Q112.G, Q97.D, R49.1
- new net N$10: Q12.G, Q13.G, Q19.D, Q20.D, Q21.G, R9.1
- new net N$101: Q128.D, Q129.D, Q131.G, Q132.G, Q159.G, R66.1
- new net N$1016: Q37.G, Q38.G, Q43.D, Q44.D, Q45.G, R22.1
- new net N$1017: Q25.D, Q26.D, Q29.G, Q30.G, Q46.G, R13.1
- new net N$102: Q132.D, Q133.D, Q142.G, R72.1
- new net N$104: Q141.D, Q142.D, Q143.G, Q156.G, R73.1
- new net N$106: Q145.D, Q146.D, Q155.G, R75.1
- new net N$108: Q143.D, Q144.D, Q147.G, R74.1
- new net N$11: Q10.D, Q11.G, Q19.G, Q9.D, R5.1
- new net N$12: Q10.G, Q6.D, Q7.D, R3.1
- new net N$124: Q73.D, Q74.D, Q76.G, Q77.G, Q90.G, R37.1
- new net N$1257: Q109.G, Q91.D, Q92.D, Q94.G, Q95.G, R46.1
- new net N$13: Q3.D, Q5.D, Q9.G, R2.1
- new net N$14: Q11.D, Q12.D, Q17.G, R6.1
- new net N$15: Q13.D, Q14.D, Q18.G, R7.1
- new net N$152: Q110.D, Q111.D, Q113.G, Q115.G, R56.1
- new net N$18: Q38.D, Q39.D, Q42.G, R19.1
- new net N$19: Q33.D, Q34.D, Q35.G, Q43.G, R17.1
- new net N$20: Q30.D, Q31.D, Q34.G, R15.1
- new net N$21: Q27.D, Q29.D, Q33.G, R14.1
- new net N$22: Q47.D, Q48.D, Q53.G, Q54.G, Q71.G, R24.1
- new net N$224: Q77.D, Q78.D, Q80.G, R39.1
- new net N$23: Q56.D, Q57.D, Q58.G, Q67.G, R27.1
- new net N$24: Q54.D, Q55.D, Q57.G, R26.1
- new net N$25: Q49.D, Q53.D, Q56.G, R25.1
- new net N$26: Q59.G, Q60.G, Q67.D, Q69.D, Q70.G, R34.1
- new net N$27: Q60.D, Q61.D, Q66.G, R29.1
- new net N$28: Q58.D, Q59.D, Q65.G, R28.1
- new net N$293: Q95.D, Q96.D, Q98.G, R48.1
- new net N$298: Q115.D, Q116.D, Q118.G, R58.1
- new net N$3: Q112.D, Q113.D, Q117.G, R57.1
- new net N$32: Q63.D, Q68.G, R36.1
- new net N$324: Q75.D, Q76.D, Q79.G, R38.1
- new net N$33: Q150.G, Q64.D, Q68.D, R76.1
- new net N$34: Q148.D, Q149.G, Q72.D, R77.1
- new net N$344: Q93.D, Q94.D, Q97.G, R47.1
- new net N$362: Q83.D, Q84.D, Q86.G, R42.1
- new net N$367: Q130.D, Q131.D, Q141.G, R67.1
- new net N$38: Q163.D, Q165.G, R86.1
- new net N$39: Q164.D, Q165.D, Q169.G, R87.1
- new net N$40: Q166.D, Q167.D, Q168.G, R88.1
- new net N$425: Q79.D, Q80.D, Q81.G, Q87.G, R40.1
- new net N$44: Q106.G, Q97.D, Q98.D, Q99.G, R49.1
- new net N$45: Q177.D, Q179.G, R94.1
- new net N$457: Q120.G, Q121.G, Q125.D, Q126.D, R63.1
- new net N$46: Q178.D, Q179.D, Q183.G, R95.1
- new net N$47: Q180.D, Q181.D, Q182.G, R96.1
- new net N$477: Q117.D, Q118.D, Q119.G, Q125.G, R59.1
- new net N$5: Q144.G, Q145.G, Q156.D, Q157.D, Q158.G, R81.1
- new net N$5234: Q82.G, Q83.G, Q87.D, Q88.D, Q89.G, R44.1
- new net N$55: Q100.G, Q101.G, Q106.D, Q107.D, Q108.G, R53.1
- new net N$615: Q101.D, Q102.D, Q104.G, R51.1
- new net N$627: Q121.D, Q122.D, Q124.G, R61.1
- new net N$7: Q15.D, Q28.G, Q8.D, R11.1
- new net N$713: Q119.D, Q120.D, Q123.G, R60.1
- new net N$715: Q100.D, Q103.G, Q99.D, R50.1
- new net N$768: Q81.D, Q82.D, Q85.G, R41.1
- new net N$9: Q1.D, Q2.D, Q22.G, Q5.G, Q6.G, R1.1
- net /CRYOUT: now also Q111.G, Q116.G, Q92.G, Q96.G; no longer Q76.G, Q77.G, Q86.G, Q88.G
- net /OP: now also Q16.G, Q166.G, Q180.G, Q72.G; no longer Q137.G, Q151.G, Q165.G, Q179.G
- net A0: now also Q128.G, Q130.G; no longer Q15.G, Q4.G
- net A1: now also Q1.G; no longer Q13.G
- net A2: now also Q25.G, Q27.G; no longer Q11.G, Q2.G
- net A3: now also Q47.G, Q49.G; no longer Q1.G, Q9.G
- net B0: now also Q148.G, Q63.G; no longer Q134.G, Q138.G
- net B0': now also Q129.G, Q133.G, Q149.D, Q150.D, R78.1; no longer Q139.D, Q140.D, Q24.G, Q8.G, R71.1
- net B1: now also Q23.G, Q4.G; no longer Q148.G, Q152.G
- net B1': now also Q2.G, Q24.D, Q28.D, R16.1; no longer Q153.D, Q154.D, Q22.G, R79.1
- net B2: now also Q163.G, Q167.G; no longer Q162.G, Q166.G
- net B2': now also Q169.D, Q26.G, Q31.G, R89.1; no longer Q167.D, Q20.G, Q6.G, R87.1
- net B3: now also Q177.G, Q181.G; no longer Q176.G, Q180.G
- net B3': now also Q183.D, Q48.G, Q55.G, R97.1; no longer Q18.G, Q181.D, Q5.G, R95.1
- net C01: now also Q14.G, Q158.D, Q159.D, Q20.G, R82.1; no longer Q39.G, Q52.D, Q60.G, Q64.D, R32.1
- net C12: now also Q21.D, Q22.D, Q39.G, Q44.G, R10.1; no longer Q38.G, Q49.D, Q57.G, Q61.D, R29.1
- net C23: now also Q45.D, Q61.G, Q69.G, R23.1; no longer Q37.G, Q54.G, Q58.D, R26.1
- net C45: now also Q102.G, Q107.G, Q89.D, Q90.D, R45.1; no longer Q101.G, Q111.D, Q116.G, Q120.D, R60.1
- net C56: now also Q109.D, Q122.G, Q126.G, R55.1; no longer Q100.G, Q113.G, Q117.D, R57.1
- net CRYIN: now also Q146.G, Q157.G; no longer Q40.G, Q63.G
- net CRYOUT: now also Q70.D, Q71.D, Q74.G, R35.1; no longer Q43.D, Q55.D, Q90.G, R23.1
- net GND: now also Q128.S, Q129.S, Q130.S, Q131.S, Q132.S, Q133.S, Q141.S, Q142.S, Q143.S, Q144.S, Q145.S, Q146.S, Q147.S, Q155.S, Q156.S, Q157.S, Q158.S, Q159.S, Q169.S, Q183.S; no longer Q134.S, Q135.S, Q136.S, Q137.S, Q138.S, Q139.S, Q140.S, Q151.S, Q152.S, Q153.S, Q154.S, Q162.S, Q176.S, Q32.S, Q36.S, Q40.S, Q50.S, Q51.S, Q52.S, Q62.S
- net N$6: now also Q15.G, Q4.D, R4.1; no longer Q162.D, Q164.G, R84.1
- net N$8: now also Q16.D, Q23.D, Q24.G, R12.1; no longer Q176.D, Q178.G, R92.1
- net N12: now also Q35.D, Q37.D, Q41.G, R18.1; no longer Q50.D, Q62.D, Q68.G, R30.1
- net OP: now also Q164.G, Q178.G, Q64.G, Q8.G; no longer Q135.G, Q149.G, Q163.G, Q177.G
- net SUM0': now also Q147.D, Q155.D, Q84.G, Q88.G, R80.1; no longer Q102.G, Q119.G, Q68.D, Q72.D, R36.1
- net SUM1: now also Q85.D, Q86.D, R43.1; no longer Q121.D, Q124.D, R61.1
- net SUM1': now also Q17.D, Q18.D, Q73.G, R8.1; no longer Q67.D, Q71.D, Q83.G, R35.1
- net SUM2: now also Q103.D, Q104.D, R52.1; no longer Q122.D, Q125.D, R62.1
- net SUM2': now also Q41.D, Q42.D, Q91.G, Q93.G, R21.1; no longer Q66.D, Q70.D, Q74.G, Q81.G, R34.1
- net SUM3: now also Q124.D, R62.1; no longer Q126.D, R63.1
- net SUM3': now also Q110.G, Q112.G, Q66.D; no longer Q69.D, Q73.G, Q79.G
- net VCC: now also R66.2, R67.2, R72.2, R73.2, R74.2, R75.2, R80.2, R81.2, R82.2, R88.2, R89.2, R96.2, R97.2; no longer R20.2, R30.2, R31.2, R32.2, R68.2, R69.2, R70.2, R71.2, R79.2, R84.2, R85.2, R92.2, R93.2
Other:
- note added: "[0] A0 B0' CRYIN -> SUM0' C01"
- note added: "[1] A1 B1' C01 -> SUM1' C12"
- note added: "[2] A2 B2' C12 -> SUM2' C23"
- note added: "[3] A3 B3' C23 -> SUM3' CRYOUT"
- note added: "[4] SUM1 CRYOUT SUM0' -> SUM1 C45"
- note added: "[5] SUM2 /CRYOUT C45 -> SUM2 C56"
- note added: "[6] SUM3 /CRYOUT -> C56 SUM3"
- moved on the sheet: C14, R1, R10, R11, R12, R13, R14, R15, R16, R17, R18, R19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

Commit message: Cleanups of PCBs
Parts:
- J1: device SparkFun-Connectors:CONN_20 -> XSNOR:PINHD-1X20/90
Changed lines of the file:
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@@
 </classes>
 <parts>
-<part name="J1" library="SparkFun-Connectors" library_urn="urn:adsk.eagle:library:513" deviceset="CONN_20" device="" package3d_urn="urn:adsk.eagle:package:38196/1"/>
+<part name="J1" library="XSNOR" library_urn="urn:adsk.eagle:library:1320997" deviceset="PINHD-1X20" device="/90" package3d_urn="urn:adsk.eagle:package:1346147/1"/>
 <part name="GND197" library="supply1" library_urn="urn:adsk.eagle:library:371" deviceset="GND" device=""/>
 <part name="P+110" library="supply1" library_urn="urn:adsk.eagle:library:371" deviceset="VCC" device=""/>
@@
 </plain>
 <instances>
-<instance part="J1" gate="G$1" x="213.36" y="363.22"/>
+<instance part="J1" gate="A" x="213.36" y="363.22"/>
 <instance part="GND197" gate="1" x="241.3" y="408.94" smashed="yes"/>
 <instance part="P+110" gate="VCC" x="241.3" y="426.72" smashed="yes">
@@
 <net name="GND" class="0">
 <segment>
-<pinref part="J1" gate="G$1" pin="20"/>
-<wire x1="226.06" y1="416.56" x2="223.52" y2="416.56" width="0.1524" layer="91"/>
+<pinref part="J1" gate="A" pin="20"/>
+<wire x1="226.06" y1="416.56" x2="210.82" y2="337.82" width="0.1524" layer="91"/>
 <label x="226.06" y="416.56" size="1.27" layer="95" xref="yes"/>
 </segment>
@@
 <net name="B0" class="0">
 <segment>
-<pinref part="J1" gate="G$1" pin="5"/>
-<wire x1="226.06" y1="378.46" x2="223.52" y2="378.46" width="0.1524" layer="91"/>
+<pinref part="J1" gate="A" pin="5"/>
+<wire x1="226.06" y1="378.46" x2="210.82" y2="375.92" width="0.1524" layer="91"/>
 <label x="226.06" y="378.46" size="1.27" layer="95" xref="yes"/>
 </segment>
@@
 </segment>
 <segment>
-<pinref part="J1" gate="G$1" pin="1"/>
-<wire x1="223.52" y1="368.3" x2="226.06" y2="368.3" width="0.1524" layer="91"/>
+<pinref part="J1" gate="A" pin="1"/>
+<wire x1="210.82" y1="386.08" x2="226.06" y2="368.3" width="0.1524" layer="91"/>
 <label x="226.06" y="368.3" size="1.27" layer="95" xref="yes"/>
 </segment>
@@
 <net name="VCC" class="0">
 <segment>
-<pinref part="J1" gate="G$1" pin="19"/>
-<wire x1="226.06" y1="414.02" x2="223.52" y2="414.02" width="0.1524" layer="91"/>
+<pinref part="J1" gate="A" pin="19"/>
+<wire x1="226.06" y1="414.02" x2="210.82" y2="340.36" width="0.1524" layer="91"/>
 <label x="226.06" y="414.02" size="1.27" layer="95" xref="yes"/>
 </segment>
@@
 <net name="B1" class="0">
 <segment>
-<pinref part="J1" gate="G$1" pin="6"/>
-<wire x1="226.06" y1="381" x2="223.52" y2="381" width="0.1524" layer="91"/>
+<pinref part="J1" gate="A" pin="6"/>
+<wire x1="226.06" y1="381" x2="210.82" y2="373.38" width="0.1524" layer="91"/>
 <label x="226.06" y="381" size="1.27" layer="95" xref="yes"/>
 </segment>
@@
 </segment>
 <segment>
-<pinref part="J1" gate="G$1" pin="2"/>
-<wire x1="226.06" y1="370.84" x2="223.52" y2="370.84" width="0.1524" layer="91"/>
+<pinref part="J1" gate="A" pin="2"/>
+<wire x1="226.06" y1="370.84" x2="210.82" y2="383.54" width="0.1524" layer="91"/>
 <label x="226.06" y="370.84" size="1.27" layer="95" xref="yes"/>
 </segment>
@@
 <net name="B2" class="0">
 <segment>
-<pinref part="J1" gate="G$1" pin="7"/>
-<wire x1="226.06" y1="383.54" x2="223.52" y2="383.54" width="0.1524" layer="91"/>
+<pinref part="J1" gate="A" pin="7"/>
+<wire x1="226.06" y1="383.54" x2="210.82" y2="370.84" width="0.1524" layer="91"/>
 <label x="226.06" y="383.54" size="1.27" layer="95" xref="yes"/>
 </segment>
@@
 </segment>
 <segment>
-<pinref part="J1" gate="G$1" pin="3"/>
-<wire x1="226.06" y1="373.38" x2="223.52" y2="373.38" width="0.1524" layer="91"/>
+<pinref part="J1" gate="A" pin="3"/>
+<wire x1="226.06" y1="373.38" x2="210.82" y2="381" width="0.1524" layer="91"/>
 <label x="226.06" y="373.38" size="1.27" layer="95" xref="yes"/>
 </segment>
@@
 <net name="B3" class="0">
 <segment>
-<pinref part="J1" gate="G$1" pin="8"/>
-<wire x1="226.06" y1="386.08" x2="223.52" y2="386.08" width="0.1524" layer="91"/>
+<pinref part="J1" gate="A" pin="8"/>
+<wire x1="226.06" y1="386.08" x2="210.82" y2="368.3" width="0.1524" layer="91"/>
 <label x="226.06" y="386.08" size="1.27" layer="95" xref="yes"/>
 </segment>
@@
 <net name="A3" class="0">
 <segment>
-<pinref part="J1" gate="G$1" pin="4"/>
-<wire x1="226.06" y1="375.92" x2="223.52" y2="375.92" width="0.1524" layer="91"/>
+<pinref part="J1" gate="A" pin="4"/>
+<wire x1="226.06" y1="375.92" x2="210.82" y2="378.46" width="0.1524" layer="91"/>
 <label x="226.06" y="375.92" size="1.27" layer="95" xref="yes"/>
 </segment>
@@
 <net name="CRYIN" class="0">
 <segment>
-<pinref part="J1" gate="G$1" pin="9"/>
-<wire x1="226.06" y1="388.62" x2="223.52" y2="388.62" width="0.1524" layer="91"/>
+<pinref part="J1" gate="A" pin="9"/>
+<wire x1="226.06" y1="388.62" x2="210.82" y2="365.76" width="0.1524" layer="91"/>
 <label x="226.06" y="388.62" size="1.27" layer="95" xref="yes"/>
 </segment>
@@
 <net name="CRYOUT" class="0">
 <segment>
-<pinref part="J1" gate="G$1" pin="14"/>
+<pinref part="J1" gate="A" pin="14"/>
 <wire x1="259.08" y1="401.32" x2="256.54" y2="401.32" width="0.1524" layer="91"/>
 <label x="259.08" y="401.32" size="1.27" layer="95" xref="yes"/>
 <pinref part="Q114" gate="NMOS" pin="G"/>
-<wire x1="256.54" y1="401.32" x2="223.52" y2="401.32" width="0.1524" layer="91"/>
+<wire x1="256.54" y1="401.32" x2="210.82" y2="353.06" width="0.1524" layer="91"/>
 <wire x1="256.54" y1="401.32" x2="256.54" y2="373.38" width="0.1524" layer="91"/>
 <wire x1="256.54" y1="373.38" x2="281.94" y2="373.38" width="0.1524" layer="91"/>
@@
 <net name="OP" class="0">
 <segment>
-<pinref part="J1" gate="G$1" pin="15"/>
+<pinref part="J1" gate="A" pin="15"/>
 <wire x1="271.78" y1="403.86" x2="269.24" y2="403.86" width="0.1524" layer="91"/>
 <label x="271.78" y="403.86" size="1.27" layer="95" xref="yes"/>
-<wire x1="269.24" y1="403.86" x2="223.52" y2="403.86" width="0.1524" layer="91"/>
+<wire x1="269.24" y1="403.86" x2="210.82" y2="350.52" width="0.1524" layer="91"/>
 <wire x1="269.24" y1="403.86" x2="269.24" y2="401.32" width="0.1524" layer="91"/>
 <junction x="269.24" y="403.86"/>
@@
 <net name="N$16" class="0">
 <segment>
-<pinref part="J1" gate="G$1" pin="16"/>
-<wire x1="226.06" y1="406.4" x2="223.52" y2="406.4" width="0.1524" layer="91"/>
+<pinref part="J1" gate="A" pin="16"/>
+<wire x1="226.06" y1="406.4" x2="210.82" y2="347.98" width="0.1524" layer="91"/>
 <label x="226.06" y="406.4" size="1.27" layer="95" xref="yes"/>
 </segment>
@@
 <net name="N$17" class="0">
 <segment>
-<pinref part="J1" gate="G$1" pin="17"/>
-<wire x1="226.06" y1="408.94" x2="223.52" y2="408.94" width="0.1524" layer="91"/>
+<pinref part="J1" gate="A" pin="17"/>
+<wire x1="226.06" y1="408.94" x2="210.82" y2="345.44" width="0.1524" layer="91"/>
 <label x="226.06" y="408.94" size="1.27" layer="95" xref="yes"/>
 </segment>
@@
 <net name="LEDPWR" class="0">
 <segment>
-<pinref part="J1" gate="G$1" pin="18"/>
-<wire x1="226.06" y1="411.48" x2="223.52" y2="411.48" width="0.1524" layer="91"/>
+<pinref part="J1" gate="A" pin="18"/>
+<wire x1="226.06" y1="411.48" x2="210.82" y2="342.9" width="0.1524" layer="91"/>
 <label x="226.06" y="411.48" size="1.27" layer="95" xref="yes"/>
 </segment>
@@
 <net name="SUM1" class="0">
 <segment>
-<pinref part="J1" gate="G$1" pin="11"/>
-<wire x1="226.06" y1="393.7" x2="223.52" y2="393.7" width="0.1524" layer="91"/>
+<pinref part="J1" gate="A" pin="11"/>
+<wire x1="226.06" y1="393.7" x2="210.82" y2="360.68" width="0.1524" layer="91"/>
 <label x="226.06" y="393.7" size="1.27" layer="95" xref="yes"/>
 </segment>
@@
 <net name="SUM2" class="0">
 <segment>
-<pinref part="J1" gate="G$1" pin="12"/>
-<wire x1="226.06" y1="396.24" x2="223.52" y2="396.24" width="0.1524" layer="91"/>
+<pinref part="J1" gate="A" pin="12"/>
+<wire x1="226.06" y1="396.24" x2="210.82" y2="358.14" width="0.1524" layer="91"/>
 <label x="226.06" y="396.24" size="1.27" layer="95" xref="yes"/>
 </segment>
@@
 <net name="SUM3" class="0">
 <segment>
-<pinref part="J1" gate="G$1" pin="13"/>
-<wire x1="226.06" y1="398.78" x2="223.52" y2="398.78" width="0.1524" layer="91"/>
+<pinref part="J1" gate="A" pin="13"/>
+<wire x1="226.06" y1="398.78" x2="210.82" y2="355.6" width="0.1524" layer="91"/>
 <label x="226.06" y="398.78" size="1.27" layer="95" xref="yes"/>
 </segment>
@@
 <wire x1="289.56" y1="353.06" x2="271.78" y2="353.06" width="0.1524" layer="91"/>
 <junction x="289.56" y="353.06"/>
-<pinref part="J1" gate="G$1" pin="10"/>
+<pinref part="J1" gate="A" pin="10"/>
 <wire x1="243.84" y1="391.16" x2="241.3" y2="391.16" width="0.1524" layer="91"/>
 <label x="243.84" y="391.16" size="1.27" layer="95" xref="yes"/>
-<wire x1="241.3" y1="391.16" x2="223.52" y2="391.16" width="0.1524" layer="91"/>
+<wire x1="241.3" y1="391.16" x2="210.82" y2="363.22" width="0.1524" layer="91"/>
 <wire x1="271.78" y1="353.06" x2="241.3" y2="353.06" width="0.1524" layer="91"/>
 <wire x1="241.3" y1="353.06" x2="241.3" y2="391.16" width="0.1524" layer="91"/>

Commit message: Updated boards with pcb template
Other:
- moved on the sheet: J1
Changed lines of the file:
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@@
 <drawing>
 <settings>
-<setting alwaysvectorfont="yes"/>
+<setting alwaysvectorfont="no"/>
 <setting verticaltext="up"/>
 </settings>
@@
 </plain>
 <instances>
-<instance part="J1" gate="A" x="213.36" y="363.22"/>
+<instance part="J1" gate="A" x="208.28" y="391.16" rot="R180"/>
 <instance part="GND197" gate="1" x="241.3" y="408.94" smashed="yes"/>
 <instance part="P+110" gate="VCC" x="241.3" y="426.72" smashed="yes">
@@
 <segment>
 <pinref part="J1" gate="A" pin="20"/>
-<wire x1="226.06" y1="416.56" x2="210.82" y2="337.82" width="0.1524" layer="91"/>
+<wire x1="226.06" y1="416.56" x2="210.82" y2="416.56" width="0.1524" layer="91"/>
 <label x="226.06" y="416.56" size="1.27" layer="95" xref="yes"/>
 </segment>
@@
 <segment>
 <pinref part="J1" gate="A" pin="5"/>
-<wire x1="226.06" y1="378.46" x2="210.82" y2="375.92" width="0.1524" layer="91"/>
+<wire x1="226.06" y1="378.46" x2="210.82" y2="378.46" width="0.1524" layer="91"/>
 <label x="226.06" y="378.46" size="1.27" layer="95" xref="yes"/>
 </segment>
@@
 <segment>
 <pinref part="J1" gate="A" pin="1"/>
-<wire x1="210.82" y1="386.08" x2="226.06" y2="368.3" width="0.1524" layer="91"/>
+<wire x1="210.82" y1="368.3" x2="226.06" y2="368.3" width="0.1524" layer="91"/>
 <label x="226.06" y="368.3" size="1.27" layer="95" xref="yes"/>
 </segment>
@@
 <segment>
 <pinref part="J1" gate="A" pin="19"/>
-<wire x1="226.06" y1="414.02" x2="210.82" y2="340.36" width="0.1524" layer="91"/>
+<wire x1="226.06" y1="414.02" x2="210.82" y2="414.02" width="0.1524" layer="91"/>
 <label x="226.06" y="414.02" size="1.27" layer="95" xref="yes"/>
 </segment>
@@
 <segment>
 <pinref part="J1" gate="A" pin="6"/>
-<wire x1="226.06" y1="381" x2="210.82" y2="373.38" width="0.1524" layer="91"/>
+<wire x1="226.06" y1="381" x2="210.82" y2="381" width="0.1524" layer="91"/>
 <label x="226.06" y="381" size="1.27" layer="95" xref="yes"/>
 </segment>
@@
 <segment>
 <pinref part="J1" gate="A" pin="2"/>
-<wire x1="226.06" y1="370.84" x2="210.82" y2="383.54" width="0.1524" layer="91"/>
+<wire x1="226.06" y1="370.84" x2="210.82" y2="370.84" width="0.1524" layer="91"/>
 <label x="226.06" y="370.84" size="1.27" layer="95" xref="yes"/>
 </segment>
@@
 <segment>
 <pinref part="J1" gate="A" pin="7"/>
-<wire x1="226.06" y1="383.54" x2="210.82" y2="370.84" width="0.1524" layer="91"/>
+<wire x1="226.06" y1="383.54" x2="210.82" y2="383.54" width="0.1524" layer="91"/>
 <label x="226.06" y="383.54" size="1.27" layer="95" xref="yes"/>
 </segment>
@@
 <segment>
 <pinref part="J1" gate="A" pin="3"/>
-<wire x1="226.06" y1="373.38" x2="210.82" y2="381" width="0.1524" layer="91"/>
+<wire x1="226.06" y1="373.38" x2="210.82" y2="373.38" width="0.1524" layer="91"/>
 <label x="226.06" y="373.38" size="1.27" layer="95" xref="yes"/>
 </segment>
@@
 <segment>
 <pinref part="J1" gate="A" pin="8"/>
-<wire x1="226.06" y1="386.08" x2="210.82" y2="368.3" width="0.1524" layer="91"/>
+<wire x1="226.06" y1="386.08" x2="210.82" y2="386.08" width="0.1524" layer="91"/>
 <label x="226.06" y="386.08" size="1.27" layer="95" xref="yes"/>
 </segment>
@@
 <segment>
 <pinref part="J1" gate="A" pin="4"/>
-<wire x1="226.06" y1="375.92" x2="210.82" y2="378.46" width="0.1524" layer="91"/>
+<wire x1="226.06" y1="375.92" x2="210.82" y2="375.92" width="0.1524" layer="91"/>
 <label x="226.06" y="375.92" size="1.27" layer="95" xref="yes"/>
 </segment>
@@
 <segment>
 <pinref part="J1" gate="A" pin="9"/>
-<wire x1="226.06" y1="388.62" x2="210.82" y2="365.76" width="0.1524" layer="91"/>
+<wire x1="226.06" y1="388.62" x2="210.82" y2="388.62" width="0.1524" layer="91"/>
 <label x="226.06" y="388.62" size="1.27" layer="95" xref="yes"/>
 </segment>
@@
 <label x="259.08" y="401.32" size="1.27" layer="95" xref="yes"/>
 <pinref part="Q114" gate="NMOS" pin="G"/>
-<wire x1="256.54" y1="401.32" x2="210.82" y2="353.06" width="0.1524" layer="91"/>
+<wire x1="256.54" y1="401.32" x2="210.82" y2="401.32" width="0.1524" layer="91"/>
 <wire x1="256.54" y1="401.32" x2="256.54" y2="373.38" width="0.1524" layer="91"/>
 <wire x1="256.54" y1="373.38" x2="281.94" y2="373.38" width="0.1524" layer="91"/>
@@
 <wire x1="271.78" y1="403.86" x2="269.24" y2="403.86" width="0.1524" layer="91"/>
 <label x="271.78" y="403.86" size="1.27" layer="95" xref="yes"/>
-<wire x1="269.24" y1="403.86" x2="210.82" y2="350.52" width="0.1524" layer="91"/>
+<wire x1="269.24" y1="403.86" x2="210.82" y2="403.86" width="0.1524" layer="91"/>
 <wire x1="269.24" y1="403.86" x2="269.24" y2="401.32" width="0.1524" layer="91"/>
 <junction x="269.24" y="403.86"/>
@@
 <segment>
 <pinref part="J1" gate="A" pin="16"/>
-<wire x1="226.06" y1="406.4" x2="210.82" y2="347.98" width="0.1524" layer="91"/>
+<wire x1="226.06" y1="406.4" x2="210.82" y2="406.4" width="0.1524" layer="91"/>
 <label x="226.06" y="406.4" size="1.27" layer="95" xref="yes"/>
 </segment>
@@
 <segment>
 <pinref part="J1" gate="A" pin="17"/>
-<wire x1="226.06" y1="408.94" x2="210.82" y2="345.44" width="0.1524" layer="91"/>
+<wire x1="226.06" y1="408.94" x2="210.82" y2="408.94" width="0.1524" layer="91"/>
 <label x="226.06" y="408.94" size="1.27" layer="95" xref="yes"/>
 </segment>
@@
 <segment>
 <pinref part="J1" gate="A" pin="18"/>
-<wire x1="226.06" y1="411.48" x2="210.82" y2="342.9" width="0.1524" layer="91"/>
+<wire x1="226.06" y1="411.48" x2="210.82" y2="411.48" width="0.1524" layer="91"/>
 <label x="226.06" y="411.48" size="1.27" layer="95" xref="yes"/>
 </segment>
@@
 <segment>
 <pinref part="J1" gate="A" pin="11"/>
-<wire x1="226.06" y1="393.7" x2="210.82" y2="360.68" width="0.1524" layer="91"/>
+<wire x1="226.06" y1="393.7" x2="210.82" y2="393.7" width="0.1524" layer="91"/>
 <label x="226.06" y="393.7" size="1.27" layer="95" xref="yes"/>
 </segment>
@@
 <segment>
 <pinref part="J1" gate="A" pin="12"/>
-<wire x1="226.06" y1="396.24" x2="210.82" y2="358.14" width="0.1524" layer="91"/>
+<wire x1="226.06" y1="396.24" x2="210.82" y2="396.24" width="0.1524" layer="91"/>
 <label x="226.06" y="396.24" size="1.27" layer="95" xref="yes"/>
 </segment>
@@
 <segment>
 <pinref part="J1" gate="A" pin="13"/>
-<wire x1="226.06" y1="398.78" x2="210.82" y2="355.6" width="0.1524" layer="91"/>
+<wire x1="226.06" y1="398.78" x2="210.82" y2="398.78" width="0.1524" layer="91"/>
 <label x="226.06" y="398.78" size="1.27" layer="95" xref="yes"/>
 </segment>
@@
 <wire x1="243.84" y1="391.16" x2="241.3" y2="391.16" width="0.1524" layer="91"/>
 <label x="243.84" y="391.16" size="1.27" layer="95" xref="yes"/>
-<wire x1="241.3" y1="391.16" x2="210.82" y2="363.22" width="0.1524" layer="91"/>
+<wire x1="241.3" y1="391.16" x2="210.82" y2="391.16" width="0.1524" layer="91"/>
 <wire x1="271.78" y1="353.06" x2="241.3" y2="353.06" width="0.1524" layer="91"/>
 <wire x1="241.3" y1="353.06" x2="241.3" y2="391.16" width="0.1524" layer="91"/>
