File: Eagle/Johnson.brd (EAGLE design)
At the start: 100 x 100 mm, 157 parts, among them Q10 310mA/60V/1.6Ω, Q100 310mA/60V/1.6Ω, Q101 310mA/60V/1.6Ω, Q102 310mA/60V/1.6Ω, Q103 310mA/60V/1.6Ω, Q104 310mA/60V/1.6Ω, Q105 310mA/60V/1.6Ω, Q106 310mA/60V/1.6Ω, Q107 310mA/60V/1.6Ω, Q108 310mA/60V/1.6Ω, Q11 310mA/60V/1.6Ω, Q12 310mA/60V/1.6Ω, Q13 310mA/60V/1.6Ω, Q14 310mA/60V/1.6Ω, Q145 310mA/60V/1.6Ω, Q146 310mA/60V/1.6Ω, Q147 310mA/60V/1.6Ω, Q148 310mA/60V/1.6Ω, Q149 310mA/60V/1.6Ω, Q15 310mA/60V/1.6Ω, Q150 310mA/60V/1.6Ω, Q151 310mA/60V/1.6Ω, Q152 310mA/60V/1.6Ω, Q153 310mA/60V/1.6Ω, Q154 310mA/60V/1.6Ω, Q155 310mA/60V/1.6Ω, Q156 310mA/60V/1.6Ω, Q157 310mA/60V/1.6Ω, Q158 310mA/60V/1.6Ω, Q159 310mA/60V/1.6Ω, Q16 310mA/60V/1.6Ω, Q160 310mA/60V/1.6Ω, Q161 310mA/60V/1.6Ω, Q162 310mA/60V/1.6Ω, Q163 310mA/60V/1.6Ω, Q164 310mA/60V/1.6Ω, Q165 310mA/60V/1.6Ω, Q166 310mA/60V/1.6Ω, Q167 310mA/60V/1.6Ω, Q168 310mA/60V/1.6Ω, Q169 310mA/60V/1.6Ω, Q17 310mA/60V/1.6Ω, Q170 310mA/60V/1.6Ω, Q171 310mA/60V/1.6Ω, Q172 310mA/60V/1.6Ω, Q173 310mA/60V/1.6Ω, Q174 310mA/60V/1.6Ω, Q175 310mA/60V/1.6Ω, Q176 310mA/60V/1.6Ω, Q177 310mA/60V/1.6Ω, Q178 310mA/60V/1.6Ω, Q179 310mA/60V/1.6Ω, Q18 310mA/60V/1.6Ω, Q180 310mA/60V/1.6Ω, Q19 310mA/60V/1.6Ω, Q20 310mA/60V/1.6Ω, Q21 310mA/60V/1.6Ω, Q22 310mA/60V/1.6Ω, Q23 310mA/60V/1.6Ω, Q24 310mA/60V/1.6Ω, Q25 310mA/60V/1.6Ω, Q26 310mA/60V/1.6Ω, Q27 310mA/60V/1.6Ω, Q28 310mA/60V/1.6Ω, Q29 310mA/60V/1.6Ω, Q3 310mA/60V/1.6Ω, Q30 310mA/60V/1.6Ω, Q31 310mA/60V/1.6Ω, Q32 310mA/60V/1.6Ω, Q33 310mA/60V/1.6Ω, Q34 310mA/60V/1.6Ω, Q35 310mA/60V/1.6Ω, Q36 310mA/60V/1.6Ω, Q37 310mA/60V/1.6Ω, Q38 310mA/60V/1.6Ω, Q4 310mA/60V/1.6Ω, Q5 310mA/60V/1.6Ω, Q6 310mA/60V/1.6Ω, Q7 310mA/60V/1.6Ω, Q73 310mA/60V/1.6Ω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

Commit message: Finished Jonsson counter pcb
Parts:
- added C1: (no value), rcl:C0805
- added Q1, Q109, Q110, Q111, Q115, Q116, Q117, Q121, Q122, Q123, Q127, Q128, Q129, Q133, Q134, Q135, Q139, Q140, Q141, Q181, Q182, Q183, Q2, Q39, Q40, Q41, Q42, Q43, Q46, Q47, Q48, Q55, Q56, Q57, Q61, Q62, Q63, Q67, Q68, Q69: 310mA/60V/1.6Ω, XSNOR:SOT23
- added R17, R18, R19, R20, R21, R23, R25, R27, R29, R31, R49, R51, R53, R55, R57: (no value), XSNOR:0805
- added SJ1, SJ10, SJ11, SJ12, SJ13, SJ14, SJ15, SJ16, SJ17, SJ2, SJ3, SJ4, SJ5, SJ6, SJ7, SJ8, SJ9: (no value), jumper:SJ_2
Connections:
- new net C0: Q42.1, SJ1.2
- new net C1: Q48.1, SJ2.2
- new net C10: Q141.1, SJ11.2
- new net C11: Q183.1, SJ12.2
- new net C2: Q57.1, SJ3.2
- new net C3: Q63.1, SJ4.2
- new net C4: Q69.1, SJ5.2
- new net C5: Q111.1, SJ6.2
- new net C6: Q117.1, SJ7.2
- new net C7: Q123.1, SJ8.2
- new net C8: Q129.1, SJ9.2
- new net C9: Q135.1, SJ10.2
- new net CLKIN: JP1.13, Q1.1, SJ13.1, SJ14.1, SJ15.1
- new net CLRIN: JP1.14, Q39.1
- new net EARLYCLR: SJ17.1
- new net N$1: SJ1.1, SJ10.1, SJ11.1, SJ12.1, SJ16.2, SJ2.1, SJ3.1, SJ4.1, SJ5.1, SJ6.1, SJ7.1, SJ8.1, SJ9.1
- new net N$17: Q2.1, SJ17.2
- new net N$3: SJ15.2, SJ16.3
- new net N$5: Q1.3, R17.1, SJ13.3, SJ14.3, SJ15.3
- new net N$6: Q2.3, Q39.3, Q43.1, R19.1
- new net O0: JP1.1, Q40.3, Q41.3, Q42.3, R18.1, SJ2.3
- new net O1: JP1.2, Q46.3, Q47.3, Q48.3, R20.1, SJ3.3
- new net O10: JP1.11, Q139.3, Q140.3, Q141.3, R55.1, SJ12.3
- new net O11: JP1.12, Q181.3, Q182.3, Q183.3, R57.1, SJ1.3
- new net O2: JP1.3, Q55.3, Q56.3, Q57.3, R23.1, SJ4.3
- new net O3: JP1.4, Q61.3, Q62.3, Q63.3, R25.1, SJ5.3
- new net O4: JP1.5, Q67.3, Q68.3, Q69.3, R27.1, SJ6.3
- new net O5: JP1.6, Q109.3, Q110.3, Q111.3, R29.1, SJ7.3
- new net O6: JP1.7, Q115.3, Q116.3, Q117.3, R31.1, SJ8.3
- new net O7: JP1.8, Q121.3, Q122.3, Q123.3, R49.1, SJ9.3
- new net O8: JP1.9, Q127.3, Q128.3, Q129.3, R51.1, SJ10.3
- new net O9: JP1.10, Q133.3, Q134.3, Q135.3, R53.1, SJ11.3
- net /CLK: now also SJ14.2
- net /Q0: now also Q115.1, Q46.1
- net /Q1: now also Q122.1, Q55.1
- net /Q2: now also Q128.1, Q61.1
- net /Q3: now also Q134.1, Q67.1
- net /Q4: now also Q109.1, Q140.1
- net /Q5: now also Q116.1, Q182.1
- net CLK: now also SJ13.2
- net CLR: now also Q43.3, R21.1
- net GND: now also C1.2, Q1.2, Q109.2, Q110.2, Q111.2, Q115.2, Q116.2, Q117.2, Q121.2, Q122.2, Q123.2, Q127.2, Q128.2, Q129.2, Q133.2, Q134.2, Q135.2, Q139.2, Q140.2, Q141.2, Q181.2, Q182.2, Q183.2, Q2.2, Q39.2, Q40.2, Q41.2, Q42.2, Q43.2, Q46.2, Q47.2, Q48.2, Q55.2, Q56.2, Q57.2, Q61.2, Q62.2, Q63.2, Q67.2, Q68.2, Q69.2, SJ16.1, SJ17.3
- net Q0: now also Q121.1, Q40.1
- net Q1: now also Q127.1, Q47.1
- net Q2: now also Q133.1, Q56.1
- net Q3: now also Q139.1, Q62.1
- net Q4: now also Q181.1, Q68.1
- net Q5: now also Q110.1, Q41.1
- net VCC: now also C1.1, R17.2, R18.2, R19.2, R20.2, R21.2, R23.2, R25.2, R27.2, R29.2, R31.2, R49.2, R51.2, R53.2, R55.2, R57.2
Routing:
- net GND: track 726.2 -> 981.6 mm, vias 48 -> 60
- net N$1: track 0.00 -> 120.5 mm, vias 0 -> 13
- net O11: track 0.00 -> 107.8 mm, vias 0 -> 1
- net O10: track 0.00 -> 102.7 mm, vias 0 -> 1
- net O9: track 0.00 -> 97.5 mm, vias 0 -> 1
- net O8: track 0.00 -> 92.3 mm, vias 0 -> 1
- net C0: track 0.00 -> 91.5 mm, vias 0 -> 2
- net O7: track 0.00 -> 86.5 mm, vias 0 -> 1
- net O6: track 0.00 -> 81.9 mm, vias 0 -> 1
- net O5: track 0.00 -> 76.7 mm, vias 0 -> 1
- net O4: track 0.00 -> 71.5 mm, vias 0 -> 1
- net EARLYCLR: track 0.00 -> 68.4 mm, vias 0 -> 2
- net O3: track 0.00 -> 66.8 mm, vias 0 -> 1
- net O0: track 0.00 -> 64.1 mm, vias 0 -> 1
- net VCC: track 555.1 -> 617.4 mm, vias 15 -> 28
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Other:
- outline, holes or cut-outs redrawn
- board text added: "0"
- board text added: "1"
- board text added: "10"
- board text added: "11"
- board text added: "2"
- board text added: "3"
- board text added: "4"
- board text added: "5"
- board text added: "6"
- board text added: "7"
- board text added: "8"
- board text added: "9"
- board text added: "Clear"
- board text added: "Clock"
- board text added: "Out0"
- board text added: "Out1"
- board text added: "Out10"
- board text added: "Out11"
- board text added: "Out2"
- board text added: "Out3"
- board text added: "Out4"
- board text added: "Out5"
- board text added: "Out6"
- board text added: "Out7"
- board text added: "Out8"
- board text added: "Out9"
- board text removed: "/CLK"
- board text removed: "CLR"
