File: Eagle/Johnson.sch (EAGLE design)
At the start: 157 parts, among them Q10 310mA/60V/1.6Ω, Q100 310mA/60V/1.6Ω, Q101 310mA/60V/1.6Ω, Q102 310mA/60V/1.6Ω, Q103 310mA/60V/1.6Ω, Q104 310mA/60V/1.6Ω, Q105 310mA/60V/1.6Ω, Q106 310mA/60V/1.6Ω, Q107 310mA/60V/1.6Ω, Q108 310mA/60V/1.6Ω, Q11 310mA/60V/1.6Ω, Q12 310mA/60V/1.6Ω, Q13 310mA/60V/1.6Ω, Q14 310mA/60V/1.6Ω, Q145 310mA/60V/1.6Ω, Q146 310mA/60V/1.6Ω, Q147 310mA/60V/1.6Ω, Q148 310mA/60V/1.6Ω, Q149 310mA/60V/1.6Ω, Q15 310mA/60V/1.6Ω, Q150 310mA/60V/1.6Ω, Q151 310mA/60V/1.6Ω, Q152 310mA/60V/1.6Ω, Q153 310mA/60V/1.6Ω, Q154 310mA/60V/1.6Ω, Q155 310mA/60V/1.6Ω, Q156 310mA/60V/1.6Ω, Q157 310mA/60V/1.6Ω, Q158 310mA/60V/1.6Ω, Q159 310mA/60V/1.6Ω, Q16 310mA/60V/1.6Ω, Q160 310mA/60V/1.6Ω, Q161 310mA/60V/1.6Ω, Q162 310mA/60V/1.6Ω, Q163 310mA/60V/1.6Ω, Q164 310mA/60V/1.6Ω, Q165 310mA/60V/1.6Ω, Q166 310mA/60V/1.6Ω, Q167 310mA/60V/1.6Ω, Q168 310mA/60V/1.6Ω, Q169 310mA/60V/1.6Ω, Q17 310mA/60V/1.6Ω, Q170 310mA/60V/1.6Ω, Q171 310mA/60V/1.6Ω, Q172 310mA/60V/1.6Ω, Q173 310mA/60V/1.6Ω, Q174 310mA/60V/1.6Ω, Q175 310mA/60V/1.6Ω, Q176 310mA/60V/1.6Ω, Q177 310mA/60V/1.6Ω, Q178 310mA/60V/1.6Ω, Q179 310mA/60V/1.6Ω, Q18 310mA/60V/1.6Ω, Q180 310mA/60V/1.6Ω, Q19 310mA/60V/1.6Ω, Q20 310mA/60V/1.6Ω, Q21 310mA/60V/1.6Ω, Q22 310mA/60V/1.6Ω, Q23 310mA/60V/1.6Ω, Q24 310mA/60V/1.6Ω, Q25 310mA/60V/1.6Ω, Q26 310mA/60V/1.6Ω, Q27 310mA/60V/1.6Ω, Q28 310mA/60V/1.6Ω, Q29 310mA/60V/1.6Ω, Q3 310mA/60V/1.6Ω, Q30 310mA/60V/1.6Ω, Q31 310mA/60V/1.6Ω, Q32 310mA/60V/1.6Ω, Q33 310mA/60V/1.6Ω, Q34 310mA/60V/1.6Ω, Q35 310mA/60V/1.6Ω, Q36 310mA/60V/1.6Ω, Q37 310mA/60V/1.6Ω, Q38 310mA/60V/1.6Ω, Q4 310mA/60V/1.6Ω, Q5 310mA/60V/1.6Ω, Q6 310mA/60V/1.6Ω, Q7 310mA/60V/1.6Ω, Q73 310mA/60V/1.6Ω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

Commit message: Finished Jonsson counter pcb
Parts:
- added C1: (no value), rcl:C-EUC0805
- added Q1, Q109, Q110, Q111, Q115, Q116, Q117, Q121, Q122, Q123, Q127, Q128, Q129, Q133, Q134, Q135, Q139, Q140, Q141, Q181, Q182, Q183, Q2, Q39, Q40, Q41, Q42, Q43, Q46, Q47, Q48, Q55, Q56, Q57, Q61, Q62, Q63, Q67, Q68, Q69: 310mA/60V/1.6Ω, XSNOR:NMOSREFLOW
- added R17, R18, R19, R20, R21, R23, R25, R27, R29, R31, R49, R51, R53, R55, R57: (no value), XSNOR:RESISTOR0805
- added SJ1, SJ10, SJ11, SJ12, SJ13, SJ14, SJ15, SJ16, SJ17, SJ2, SJ3, SJ4, SJ5, SJ6, SJ7, SJ8, SJ9: (no value), jumper:SJ2W
Connections:
- new net C0: Q42.G, SJ1.2
- new net C1: Q48.G, SJ2.2
- new net C10: Q141.G, SJ11.2
- new net C11: Q183.G, SJ12.2
- new net C2: Q57.G, SJ3.2
- new net C3: Q63.G, SJ4.2
- new net C4: Q69.G, SJ5.2
- new net C5: Q111.G, SJ6.2
- new net C6: Q117.G, SJ7.2
- new net C7: Q123.G, SJ8.2
- new net C8: Q129.G, SJ9.2
- new net C9: Q135.G, SJ10.2
- new net CLKIN: JP1.13, Q1.G, SJ13.1, SJ14.1, SJ15.1
- new net CLRIN: JP1.14, Q39.G
- new net EARLYCLR: SJ17.1
- new net N$1: SJ1.1, SJ10.1, SJ11.1, SJ12.1, SJ16.2, SJ2.1, SJ3.1, SJ4.1, SJ5.1, SJ6.1, SJ7.1, SJ8.1, SJ9.1
- new net N$17: Q2.G, SJ17.2
- new net N$3: SJ15.2, SJ16.3
- new net N$5: Q1.D, R17.1, SJ13.3, SJ14.3, SJ15.3
- new net N$6: Q2.D, Q39.D, Q43.G, R19.1
- new net O0: JP1.1, Q40.D, Q41.D, Q42.D, R18.1, SJ2.3
- new net O1: JP1.2, Q46.D, Q47.D, Q48.D, R20.1, SJ3.3
- new net O10: JP1.11, Q139.D, Q140.D, Q141.D, R55.1, SJ12.3
- new net O11: JP1.12, Q181.D, Q182.D, Q183.D, R57.1, SJ1.3
- new net O2: JP1.3, Q55.D, Q56.D, Q57.D, R23.1, SJ4.3
- new net O3: JP1.4, Q61.D, Q62.D, Q63.D, R25.1, SJ5.3
- new net O4: JP1.5, Q67.D, Q68.D, Q69.D, R27.1, SJ6.3
- new net O5: JP1.6, Q109.D, Q110.D, Q111.D, R29.1, SJ7.3
- new net O6: JP1.7, Q115.D, Q116.D, Q117.D, R31.1, SJ8.3
- new net O7: JP1.8, Q121.D, Q122.D, Q123.D, R49.1, SJ9.3
- new net O8: JP1.9, Q127.D, Q128.D, Q129.D, R51.1, SJ10.3
- new net O9: JP1.10, Q133.D, Q134.D, Q135.D, R53.1, SJ11.3
- net /CLK: now also SJ14.2
- net /Q0: now also Q115.G, Q46.G
- net /Q1: now also Q122.G, Q55.G
- net /Q2: now also Q128.G, Q61.G
- net /Q3: now also Q134.G, Q67.G
- net /Q4: now also Q109.G, Q140.G
- net /Q5: now also Q116.G, Q182.G
- net CLK: now also SJ13.2
- net CLR: now also Q43.D, R21.1
- net GND: now also C1.2, Q1.S, Q109.S, Q110.S, Q111.S, Q115.S, Q116.S, Q117.S, Q121.S, Q122.S, Q123.S, Q127.S, Q128.S, Q129.S, Q133.S, Q134.S, Q135.S, Q139.S, Q140.S, Q141.S, Q181.S, Q182.S, Q183.S, Q2.S, Q39.S, Q40.S, Q41.S, Q42.S, Q43.S, Q46.S, Q47.S, Q48.S, Q55.S, Q56.S, Q57.S, Q61.S, Q62.S, Q63.S, Q67.S, Q68.S, Q69.S, SJ16.1, SJ17.3
- net Q0: now also Q121.G, Q40.G
- net Q1: now also Q127.G, Q47.G
- net Q2: now also Q133.G, Q56.G
- net Q3: now also Q139.G, Q62.G
- net Q4: now also Q181.G, Q68.G
- net Q5: now also Q110.G, Q41.G
- net VCC: now also C1.1, R17.2, R18.2, R19.2, R20.2, R21.2, R23.2, R25.2, R27.2, R29.2, R31.2, R49.2, R51.2, R53.2, R55.2, R57.2
Other:
- moved on the sheet: Q10, Q100, Q101, Q102, Q103, Q104, Q105, Q106, Q107, Q108, Q11, Q12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
