File: Eagle/AddSub.brd (EAGLE design)
At the start: 100 x 100 mm, 238 parts, among them Q1 310mA/60V/1.6Ω, Q10 310mA/60V/1.6Ω, Q100 310mA/60V/1.6Ω, Q101 310mA/60V/1.6Ω, Q102 310mA/60V/1.6Ω, Q103 310mA/60V/1.6Ω, Q104 310mA/60V/1.6Ω, Q105 310mA/60V/1.6Ω, Q106 310mA/60V/1.6Ω, Q107 310mA/60V/1.6Ω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

Commit message: Cleanup
Routing:
- net GND: track 1079.8 -> 1065.0 mm
- net C56: track 40.1 -> 42.6 mm
- net N$3: track 19.1 -> 20.7 mm
- net N$298: track 16.1 -> 15.5 mm
